Commit message: Add the properties: mass and inertia to mockingbird

File: rotors_description/urdf/mockingbird.xacro (robot description, xacro)
@@ -24,19 +24,19 @@
   <xacro:property name="mesh_file_core" value="package://rotors_description/meshes/mockingbird_core.dae" />
   <xacro:property name="mesh_file_rotor_unit" value="package://rotors_description/meshes/mockingbird_rotorunit.dae" />
-  <xacro:property name="mass_core" value="0.5" /> <!-- [kg] -->
-  <xacro:property name="mass_rotor_unit" value="0.1" /> <!-- [kg] -->
-  <xacro:property name="body_width" value="0.1" /> <!-- [m] -->
-  <xacro:property name="body_height" value="0.16" /> <!-- [m] -->
-  <xacro:property name="mass_rotor" value="0.005" /> <!-- [kg] -->
-  <xacro:property name="arm_length" value="0.256" /> <!-- [m] -->
-  <xacro:property name="rotor_offset_top" value="0.042" /> <!-- [m] -->
+  <xacro:property name="mass_core" value="1.63543" /> <!-- [kg] -->
+  <xacro:property name="mass_rotor_unit" value="0.097214  " /> <!-- [kg] -->
+  <xacro:property name="body_width" value="0.22" /> <!-- [m] -->
+  <xacro:property name="body_height" value="0.13" /> <!-- [m] -->
+  <xacro:property name="mass_rotor" value="0.004" /> <!-- [kg] -->
+  <xacro:property name="arm_length" value="0.270" /> <!-- [m] -->
+  <xacro:property name="rotor_offset_top" value="0.038" /> <!-- [m] -->
   <xacro:property name="radius_rotor" value="0.0765" /> <!-- [m] -->
-  <xacro:property name="motor_constant" value="8.54858e-06" /> <!-- [kg m/s^2] -->
+  <xacro:property name="motor_constant" value="${1.2*8.54858e-06}" /> <!-- [kg m/s^2] -->
   <xacro:property name="moment_constant" value="0.016" /> <!-- [m] -->
   <xacro:property name="time_constant_up" value="0.0125" /> <!-- [s] -->
   <xacro:property name="time_constant_down" value="0.025" /> <!-- [s] -->
   <xacro:property name="max_rot_velocity" value="838" /> <!-- [rad/s] --> <!-- so that it produce 1 kg thrust -->
-  <xacro:property name="lower_limit_revolute" value="0" /> <!-- properties of the revolute joint of the tilted axis -->
-  <xacro:property name="upper_limit_revolute" value="0" /> <!-- properties of the revolute joint of the tilted axis -->
+  <xacro:property name="lower_limit_revolute" value="${0-0.3}" /> <!-- properties of the revolute joint of the tilted axis -->
+  <xacro:property name="upper_limit_revolute" value="${0+0.3}" /> <!-- properties of the revolute joint of the tilted axis -->
   <xacro:property name="effort_revolute" value="1000" /> <!-- properties of the revolute joint of the tilted axis -->
   <xacro:property name="velocity_revolute" value="4" /> <!-- properties of the revolute joint of the tilted axis -->
@@ -45,7 +45,11 @@
   <xacro:property name="rotor_drag_coefficient" value="8.06428e-05" />
   <xacro:property name="rolling_moment_coefficient" value="0.000001" />
-  <!-- Property Blocks -->
+  <!-- Property Blocks UPDATE:20.12.16-->
   <xacro:property name="body_inertia">
-    <inertia ixx="0.0347563" ixy="0.0" ixz="0.0" iyy="0.0458929" iyz="0.0" izz="0.0977" /> <!-- [kg m^2] [kg m^2] [kg m^2] [kg m^2] [kg m^2] [kg m^2] -->
+    <inertia ixx="0.01264185265" ixy="0.000044900117" ixz="0.00012360562" iyy="0.0127500516" iyz="-0.000018183082" izz="0.02307491809" /> <!-- [kg m^2] [kg m^2] [kg m^2] [kg m^2] [kg m^2] [kg m^2] -->
+  </xacro:property>
+  <!-- Rotor unit inertia without the propellor -->
+  <xacro:property name="rotor_unit_inertia">
+    <inertia ixx="0.000247268773" ixy="0" ixz="0" iyy="0.0003322455" iyz="0" izz="0.0002478588" /> <!-- [kg m^2] [kg m^2] [kg m^2] [kg m^2] [kg m^2] [kg m^2] -->
   </xacro:property>
   <!-- inertia of a single rotor, assuming it is a cuboid. Height=3mm, width=15mm -->
@@ -79,5 +83,5 @@
     mesh_rotor_unit="${mesh_file_rotor_unit}">
     <origin xyz="${cos30*arm_length} ${sin30*arm_length} 0" rpy="0 0 0.52359877559" />
-    <xacro:insert_block name="rotor_inertia" />
+    <xacro:insert_block name="rotor_unit_inertia" />
   </xacro:rotor_unit>
   <xacro:rotor_unit
@@ -93,5 +97,5 @@
     mesh_rotor_unit="${mesh_file_rotor_unit}">
     <origin xyz="0 ${arm_length} 0" rpy="0 0 1.57079632679" />
-    <xacro:insert_block name="rotor_inertia" />
+    <xacro:insert_block name="rotor_unit_inertia" />
   </xacro:rotor_unit>
   <xacro:rotor_unit
@@ -107,5 +111,5 @@
     mesh_rotor_unit="${mesh_file_rotor_unit}">
     <origin xyz="-${cos30*arm_length} ${sin30*arm_length} 0" rpy="0 0 2.61799387799" />
-    <xacro:insert_block name="rotor_inertia" />
+    <xacro:insert_block name="rotor_unit_inertia" />
   </xacro:rotor_unit>
   <xacro:rotor_unit
@@ -121,5 +125,5 @@
     mesh_rotor_unit="${mesh_file_rotor_unit}">
     <origin xyz="-${cos30*arm_length} -${sin30*arm_length} 0" rpy="0 0 3.66519142919" />
-    <xacro:insert_block name="rotor_inertia" />
+    <xacro:insert_block name="rotor_unit_inertia" />
   </xacro:rotor_unit>
   <xacro:rotor_unit
@@ -135,5 +139,5 @@
     mesh_rotor_unit="${mesh_file_rotor_unit}">
     <origin xyz="0 -${arm_length} 0" rpy="0 0 4.71238898038" />
-    <xacro:insert_block name="rotor_inertia" />
+    <xacro:insert_block name="rotor_unit_inertia" />
   </xacro:rotor_unit>
   <xacro:rotor_unit
@@ -149,5 +153,5 @@
     mesh_rotor_unit="${mesh_file_rotor_unit}">
     <origin xyz="${cos30*arm_length} -${sin30*arm_length} 0" rpy="0 0 5.75958653158" />
-    <xacro:insert_block name="rotor_inertia" />
+    <xacro:insert_block name="rotor_unit_inertia" />
   </xacro:rotor_unit>
   <!-- Instantiate rotors -->
