Commit message: All most fixed the problem with the newly attached controller of the servos

File: rotors_description/urdf/mockingbird_base.xacro (robot description, xacro)
@@ -22,4 +22,10 @@
   <!-- Instantiate a controller. -->
   <xacro:controller_plugin_macro namespace="${namespace}" imu_sub_topic="imu" />
+  <!-- Try to add controller to servo motors -->
+  <gazebo>
+    <plugin name="gazebo_ros_control" filename="libgazebo_ros_control.so">
+      <robotNamespace>${namespace}</robotNamespace>
+    </plugin>
+  </gazebo>
   <xacro:if value="$(arg enable_mavlink_interface)">
     <!-- Instantiate mavlink telemetry interface. -->

File: rotors_description/urdf/multirotor_base.xacro (robot description, xacro)
@@ -135,5 +135,5 @@
   <xacro:macro name="rotor_unit"
     params="robot_namespace suffix mass_rotor_unit parent motor_number lower_limit upper_limit effort velocity mesh_rotor_unit *origin *inertia">
-    <joint name="${robot_namespace}/rotor_unit_${motor_number}_revolutejoint" type="revolute">
+    <joint name="${robot_namespace}/rotor_unit_${motor_number}_joint" type="revolute">
       <xacro:insert_block name="origin" />
       <axis xyz="1 0 0" />
@@ -146,5 +146,5 @@
     <transmission name="${robot_namespace}/rotor_unit_${motor_number}_trans">
       <type>transmission_interface/SimpleTransmission</type>
-        <joint name="${robot_namespace}/rotor_unit_${motor_number}_revolutejoint">
+        <joint name="${robot_namespace}/rotor_unit_${motor_number}_joint">
           <hardwareInterface>EffortJointInterface</hardwareInterface>
         </joint>

Commit message: Last save before branch for testing the nameconvention of rrbot

File: rotors_description/urdf/mockingbird_base.xacro (robot description, xacro)
@@ -26,4 +26,5 @@
     <plugin name="gazebo_ros_control" filename="libgazebo_ros_control.so">
       <robotNamespace>${namespace}</robotNamespace>
+      <robotParam>${namespace}/robot_description</robotParam>
     </plugin>
   </gazebo>

File: rotors_description/urdf/multirotor_base.xacro (robot description, xacro)
@@ -135,5 +135,5 @@
   <xacro:macro name="rotor_unit"
     params="robot_namespace suffix mass_rotor_unit parent motor_number lower_limit upper_limit effort velocity mesh_rotor_unit *origin *inertia">
-    <joint name="${robot_namespace}/rotor_unit_${motor_number}_joint" type="revolute">
+    <joint name="${robot_namespace}/rotor_unit_${motor_number}_revolutejoint" type="revolute">
       <xacro:insert_block name="origin" />
       <axis xyz="1 0 0" />
@@ -144,14 +144,4 @@
       <child link="${robot_namespace}/rotor_unit_${motor_number}" />
     </joint>
-    <transmission name="${robot_namespace}/rotor_unit_${motor_number}_trans">
-      <type>transmission_interface/SimpleTransmission</type>
-        <joint name="${robot_namespace}/rotor_unit_${motor_number}_joint">
-          <hardwareInterface>EffortJointInterface</hardwareInterface>
-        </joint>
-        <actuator name="${robot_namespace}/rotor_unit_${motor_number}_tiltmotor">
-          <hardwareInterface>EffortJointInterface</hardwareInterface>
-          <mechanicalReduction>1</mechanicalReduction>
-        </actuator>
-    </transmission>
     <link name="${robot_namespace}/rotor_unit_${motor_number}">
       <inertial>
@@ -172,4 +162,14 @@
       </collision>
     </link>
+    <transmission name="${robot_namespace}/rotor_unit_${motor_number}_trans">
+      <type>transmission_interface/SimpleTransmission</type>
+        <joint name="${robot_namespace}/rotor_unit_${motor_number}_revolutejoint">
+          <hardwareInterface>EffortJointInterface</hardwareInterface>
+        </joint>
+        <actuator name="${robot_namespace}/rotor_unit_${motor_number}_tiltmotor">
+          <hardwareInterface>EffortJointInterface</hardwareInterface>
+          <mechanicalReduction>1</mechanicalReduction>
+        </actuator>
+    </transmission>
   </xacro:macro>
 </robot>

Commit message: restore changes to state before branching

File: rotors_description/urdf/mockingbird_base.xacro (robot description, xacro)
@@ -26,5 +26,6 @@
     <plugin name="gazebo_ros_control" filename="libgazebo_ros_control.so">
       <robotNamespace>${namespace}</robotNamespace>
-      <robotParam>${namespace}/robot_description</robotParam>
+       <robotSimType>gazebo_ros_control/DefaultRobotHWSim</robotSimType>
+      <!-- <robotParam>${namespace}/robot_description</robotParam> -->
     </plugin>
   </gazebo>

File: rotors_description/urdf/multirotor_base.xacro (robot description, xacro)
@@ -135,5 +135,5 @@
   <xacro:macro name="rotor_unit"
     params="robot_namespace suffix mass_rotor_unit parent motor_number lower_limit upper_limit effort velocity mesh_rotor_unit *origin *inertia">
-    <joint name="${robot_namespace}/rotor_unit_${motor_number}_revolutejoint" type="revolute">
+    <joint name="${namespace}/rotor_unit_${motor_number}_revolutejoint" type="revolute">
       <xacro:insert_block name="origin" />
       <axis xyz="1 0 0" />
@@ -142,7 +142,7 @@
       <!-- <limit effort="2000" velocity="${max_rot_velocity}" /> -->
       <parent link="${parent}" />
-      <child link="${robot_namespace}/rotor_unit_${motor_number}" />
+      <child link="${namespace}/rotor_unit_${motor_number}" />
     </joint>
-    <link name="${robot_namespace}/rotor_unit_${motor_number}">
+    <link name="${namespace}/rotor_unit_${motor_number}">
       <inertial>
         <mass value="${mass_rotor_unit}" /> <!-- [kg] -->
@@ -162,10 +162,10 @@
       </collision>
     </link>
-    <transmission name="${robot_namespace}/rotor_unit_${motor_number}_trans">
+    <transmission name="${namespace}/rotor_unit_${motor_number}_trans">
       <type>transmission_interface/SimpleTransmission</type>
-        <joint name="${robot_namespace}/rotor_unit_${motor_number}_revolutejoint">
+        <joint name="${namespace}/rotor_unit_${motor_number}_revolutejoint">
           <hardwareInterface>EffortJointInterface</hardwareInterface>
         </joint>
-        <actuator name="${robot_namespace}/rotor_unit_${motor_number}_tiltmotor">
+        <actuator name="${namespace}/rotor_unit_${motor_number}_tiltmotor">
           <hardwareInterface>EffortJointInterface</hardwareInterface>
           <mechanicalReduction>1</mechanicalReduction>

Commit message: solved the problem, tilting units could no be positioned

File: rotors_description/urdf/mockingbird_base.xacro (robot description, xacro)
@@ -26,7 +26,7 @@
     <plugin name="gazebo_ros_control" filename="libgazebo_ros_control.so">
       <robotNamespace>${namespace}/mockingbird</robotNamespace>
-       <robotSimType>gazebo_ros_control/DefaultRobotHWSim</robotSimType>
+       <!-- <robotSimType>gazebo_ros_control/DefaultRobotHWSim</robotSimType> -->
        <!-- <linkName>${namespace}/base_link</linkName> -->
-      <!-- <robotParam>${namespace}/robot_description</robotParam> -->
+      <robotParam>robot_description</robotParam>
     </plugin>
   </gazebo>

File: rotors_description/urdf/multirotor_base.xacro (robot description, xacro)
@@ -135,5 +135,5 @@
   <xacro:macro name="rotor_unit"
     params="robot_namespace suffix mass_rotor_unit parent motor_number lower_limit upper_limit effort velocity mesh_rotor_unit *origin *inertia">
-    <joint name="${namespace}/rotor_unit_${motor_number}_revolutejoint" type="revolute">
+    <joint name="rotor_unit_${motor_number}_revolutejoint" type="revolute">
       <xacro:insert_block name="origin" />
       <axis xyz="1 0 0" />
@@ -162,10 +162,10 @@
       </collision>
     </link>
-    <transmission name="${namespace}/rotor_unit_${motor_number}_trans">
+    <transmission name="rotor_unit_${motor_number}_trans">
       <type>transmission_interface/SimpleTransmission</type>
-        <joint name="${namespace}/rotor_unit_${motor_number}_revolutejoint">
+        <joint name="rotor_unit_${motor_number}_revolutejoint">
           <hardwareInterface>EffortJointInterface</hardwareInterface>
         </joint>
-        <actuator name="${namespace}/rotor_unit_${motor_number}_tiltmotor">
+        <actuator name="rotor_unit_${motor_number}_tiltmotor">
           <hardwareInterface>EffortJointInterface</hardwareInterface>
           <mechanicalReduction>1</mechanicalReduction>
