Commit message: Updated the specification of mockingbird

File: rotors_description/urdf/mockingbird_without_rotorguard.xacro (robot description, xacro)
@@ -22,9 +22,10 @@
     <xacro:property name="use_mesh_file_core" value="true"/>
     <xacro:property name="use_mesh_file_rotor_unit" value="true"/>
-    <xacro:property name="mesh_file_core" value="package://rotors_description/meshes/mockingbird_core.dae"/>
+    <xacro:property name="mesh_file_core" value="package://rotors_description/meshes/mockingbird_core_light.dae"/>
     <xacro:property name="mesh_file_rotor_unit" value="package://rotors_description/meshes/mockingbird_rotorunit.dae"/>
-    <xacro:property name="mass_core" value="1.63543"/>
+    <!-- <xacro:property name="mesh_file_rotor_unit" value="package://rotors_description/meshes/mockingbird_rotorunit_wo_rotorguard.dae"/> -->
+    <xacro:property name="mass_core" value="1.16"/>
     <!-- [kg] -->
-    <xacro:property name="mass_rotor_unit" value="0.097214  "/>
+    <xacro:property name="mass_rotor_unit" value="0.112"/>
     <!-- [kg] -->
     <xacro:property name="body_width" value="0.22"/>
@@ -32,11 +33,11 @@
     <xacro:property name="body_height" value="0.13"/>
     <!-- [m] -->
-    <xacro:property name="mass_rotor" value="0.004"/>
+    <xacro:property name="mass_rotor" value="0.015"/>
     <!-- [kg] -->
-    <xacro:property name="arm_length" value="0.270"/>
-    <!-- [m] -->
-    <xacro:property name="rotor_offset_top" value="0.038"/>
-    <!-- [m] -->
-    <xacro:property name="radius_rotor" value="0.0765"/>
+    <xacro:property name="arm_length" value="${0.75/2}"/>
+    <!-- [m] -->
+    <xacro:property name="rotor_offset_top" value="0.055"/>
+    <!-- [m] -->
+    <xacro:property name="radius_rotor" value="0.12"/>
     <!-- [m] -->
     <xacro:property name="motor_constant" value="${1.2*8.54858e-06}"/>
@@ -63,12 +64,12 @@
     <xacro:property name="rotor_drag_coefficient" value="8.06428e-05"/>
     <xacro:property name="rolling_moment_coefficient" value="0.000001"/>
-    <!-- Property Blocks UPDATE:20.12.16-->
+    <!-- Property Blocks UPDATE:29.02.17-->
     <xacro:property name="body_inertia">
-        <inertia ixx="0.01264185265" ixy="0.000044900117" ixz="0.00012360562" iyy="0.0127500516" iyz="-0.000018183082" izz="0.02307491809"/>
+        <inertia ixx="0.024203" ixy="0.00004500117" ixz="0.00018060562" iyy="0.02484" iyz="-0.000018183082" izz="0.045521"/>
         <!-- [kg m^2] [kg m^2] [kg m^2] [kg m^2] [kg m^2] [kg m^2] -->
     </xacro:property>
     <!-- Rotor unit inertia without the propellor -->
     <xacro:property name="rotor_unit_inertia">
-        <inertia ixx="0.000247268773" ixy="0" ixz="0" iyy="0.0003322455" iyz="0" izz="0.0002478588"/>
+        <inertia ixx="0.000084" ixy="0" ixz="0" iyy="0.000084" iyz="0" izz="0.000015"/>
         <!-- [kg m^2] [kg m^2] [kg m^2] [kg m^2] [kg m^2] [kg m^2] -->
     </xacro:property>
