Commit message: Added color to our modell, Added MSF (Flight with IMU) to the simulation

File: rotors_description/urdf/firefly.xacro (robot description, xacro)
@@ -52,4 +52,5 @@
     robot_namespace="${namespace}"
     mass="${mass}"
+    color="Turquoise"
     body_width="${body_width}"
     body_height="${body_height}"

File: rotors_description/urdf/mockingbird_base.xacro (robot description, xacro)
@@ -25,5 +25,5 @@
     <gazebo>
         <plugin name="gazebo_ros_control" filename="libgazebo_ros_control.so">
-            <robotNamespace>${namespace}/mockingbird</robotNamespace>
+            <robotNamespace>${namespace}</robotNamespace>
             <!-- <robotSimType>gazebo_ros_control/DefaultRobotHWSim</robotSimType> -->
             <!-- <linkName>${namespace}/base_link</linkName> -->

File: rotors_description/urdf/mockingbird_without_rotorguard.xacro (robot description, xacro)
@@ -26,4 +26,5 @@
     <!-- <xacro:property name="mesh_file_rotor_unit" value="package://rotors_description/meshes/mockingbird_rotorunit_wo_rotorguard.dae"/> -->
     <xacro:property name="mass_core" value="1.16"/>
+    <!-- <xacro:property name="mass_core" value="2.16"/> -->
     <!-- [kg] -->
     <xacro:property name="mass_rotor_unit" value="0.112"/>
@@ -42,4 +43,5 @@
     <!-- [m] -->
     <xacro:property name="motor_constant" value="${1.2*8.54858e-06}"/>
+    <!-- <xacro:property name="motor_constant" value="${4.44e-05}"/> -->
     <!-- [kg m/s^2] -->
     <xacro:property name="moment_constant" value="0.016"/>
@@ -50,9 +52,10 @@
     <!-- [s] -->
     <xacro:property name="max_rot_velocity" value="838"/>
+    <!-- <xacro:property name="max_rot_velocity" value="171.1"/> -->
     <!-- [rad/s] -->
     <!-- so that it produce 1 kg thrust -->
-    <xacro:property name="lower_limit_revolute" value="${0-0.3}"/>
+    <xacro:property name="lower_limit_revolute" value="${0-3}"/>
     <!-- properties of the revolute joint of the tilted axis -->
-    <xacro:property name="upper_limit_revolute" value="${0+0.3}"/>
+    <xacro:property name="upper_limit_revolute" value="${0+3}"/>
     <!-- properties of the revolute joint of the tilted axis -->
     <xacro:property name="effort_revolute" value="1000"/>
@@ -81,5 +84,5 @@
     <xacro:include filename="$(find rotors_description)/urdf/multirotor_base.xacro"/>
     <!-- Instantiate multirotor_base_macro once -->
-    <xacro:multirotor_base_macro robot_namespace="${namespace}" mass="${mass_core}" body_width="${body_width}" body_height="${body_height}" use_mesh_file="${use_mesh_file_core}" mesh_file="${mesh_file_core}">
+    <xacro:multirotor_base_macro robot_namespace="${namespace}" mass="${mass_core}" color="ZincYellow" body_width="${body_width}" body_height="${body_height}" use_mesh_file="${use_mesh_file_core}" mesh_file="${mesh_file_core}">
         <xacro:insert_block name="body_inertia"/>
     </xacro:multirotor_base_macro>
@@ -95,5 +98,6 @@
         effort="${effort_revolute}"
         velocity="${velocity_revolute}"
-        mesh_rotor_unit="${mesh_file_rotor_unit}">
+        mesh_rotor_unit="${mesh_file_rotor_unit}"
+        color="Orange">
         <origin xyz="${cos30*arm_length} ${sin30*arm_length} 0" rpy="0 0 0.52359877559"/>
         <xacro:insert_block name="rotor_unit_inertia"/>
@@ -109,5 +113,6 @@
         effort="${effort_revolute}"
         velocity="${velocity_revolute}"
-        mesh_rotor_unit="${mesh_file_rotor_unit}">
+        mesh_rotor_unit="${mesh_file_rotor_unit}"
+        color="Grey">
         <origin xyz="0 ${arm_length} 0" rpy="0 0 1.57079632679"/>
         <xacro:insert_block name="rotor_unit_inertia"/>
@@ -123,5 +128,6 @@
         effort="${effort_revolute}"
         velocity="${velocity_revolute}"
-        mesh_rotor_unit="${mesh_file_rotor_unit}">
+        mesh_rotor_unit="${mesh_file_rotor_unit}"
+        color="Grey">
         <origin xyz="-${cos30*arm_length} ${sin30*arm_length} 0" rpy="0 0 2.61799387799"/>
         <xacro:insert_block name="rotor_unit_inertia"/>
@@ -137,5 +143,6 @@
         effort="${effort_revolute}"
         velocity="${velocity_revolute}"
-        mesh_rotor_unit="${mesh_file_rotor_unit}">
+        mesh_rotor_unit="${mesh_file_rotor_unit}"
+        color="Grey">
         <origin xyz="-${cos30*arm_length} -${sin30*arm_length} 0" rpy="0 0 3.66519142919"/>
         <xacro:insert_block name="rotor_unit_inertia"/>
@@ -151,5 +158,6 @@
         effort="${effort_revolute}"
         velocity="${velocity_revolute}"
-        mesh_rotor_unit="${mesh_file_rotor_unit}">
+        mesh_rotor_unit="${mesh_file_rotor_unit}"
+        color="Grey">
         <origin xyz="0 -${arm_length} 0" rpy="0 0 4.71238898038"/>
         <xacro:insert_block name="rotor_unit_inertia"/>
@@ -165,5 +173,6 @@
         effort="${effort_revolute}"
         velocity="${velocity_revolute}"
-        mesh_rotor_unit="${mesh_file_rotor_unit}">
+        mesh_rotor_unit="${mesh_file_rotor_unit}"
+        color="Orange">
         <origin xyz="${cos30*arm_length} -${sin30*arm_length} 0" rpy="0 0 5.75958653158"/>
         <xacro:insert_block name="rotor_unit_inertia"/>
@@ -227,5 +236,5 @@
         rotor_drag_coefficient="${rotor_drag_coefficient}"
         rolling_moment_coefficient="${rolling_moment_coefficient}"
-        color="Blue"
+        color="Red"
         use_own_mesh="false"
         mesh="">
@@ -269,5 +278,5 @@
         rotor_drag_coefficient="${rotor_drag_coefficient}"
         rolling_moment_coefficient="${rolling_moment_coefficient}"
-        color="Blue"
+        color="Red"
         use_own_mesh="false"
         mesh="">
@@ -290,5 +299,5 @@
         rotor_drag_coefficient="${rotor_drag_coefficient}"
         rolling_moment_coefficient="${rolling_moment_coefficient}"
-        color="Red"
+        color="Blue"
         use_own_mesh="false"
         mesh="">

File: rotors_description/urdf/multirotor_base.xacro (robot description, xacro)
@@ -33,5 +33,5 @@
   <!-- Main multirotor link -->
   <xacro:macro name="multirotor_base_macro"
-    params="robot_namespace mass body_width body_height use_mesh_file mesh_file *inertia">
+    params="robot_namespace mass color body_width body_height use_mesh_file mesh_file *inertia">
     <link name="${robot_namespace}/base_link"></link>
     <joint name="${robot_namespace}/base_joint" type="fixed">
@@ -64,4 +64,7 @@
       </collision>
     </link>
+    <gazebo reference="${robot_namespace}/base_link">
+      <material>Gazebo/${color}</material>
+    </gazebo>
     <!-- attach multirotor_base_plugin to the base_link -->
     <gazebo>
@@ -134,5 +137,5 @@
   <!-- Tilting rotorunit link and joint -->
   <xacro:macro name="rotor_unit"
-    params="robot_namespace suffix mass_rotor_unit parent motor_number lower_limit upper_limit effort velocity mesh_rotor_unit *origin *inertia">
+    params="robot_namespace suffix mass_rotor_unit parent motor_number lower_limit upper_limit effort velocity mesh_rotor_unit color *origin *inertia">
     <joint name="rotor_unit_${motor_number}_revolutejoint" type="revolute">
       <xacro:insert_block name="origin" />
@@ -172,4 +175,7 @@
         </actuator>
     </transmission>
+    <gazebo reference="${robot_namespace}/rotor_unit_${motor_number}">
+      <material>Gazebo/${color}</material>
+    </gazebo>
   </xacro:macro>
 </robot>
